File: embedded_system_project_kicad/embedded_system_project.kicad_pcb (KiCad board)
At the start: 2 copper layers, 56 parts, among them Q1 2N2222A, U1 AMS1117CD-3.3

Commit message: Updated repo
Parts:
- removed MIC1: INMP441, inmp441:inmp441
- removed U1: AMS1117CD-3.3, Package_TO_SOT_SMD:TO-252-3_TabPin2
- added C14: 1000 microF, Capacitor_THT:CP_Axial_L10.0mm_D4.5mm_P15.00mm_Horizontal, F.Cu at (109.2, 87.4)
- added R14: 1k, Resistor_THT:R_Axial_DIN0207_L6.3mm_D2.5mm_P7.62mm_Horizontal, F.Cu at (96.8, 77.6)
- added REG2: LM1085-3.3, LM1085IT-3.3:TO254P1054X470X1955-3, F.Cu at (109.1, 75.8)
- 1N914: value D -> D2; footprint Diode_THT:D_5KPW_P12.70mm_Horizontal -> 1N914:DIOAD753W49L380D172B
- D1: value 1N4007W -> 1N4007; footprint Diode_SMD:D_1206_3216Metric_Pad1.42x1.75mm_HandSolder -> Diode_THT:D_DO-41_SOD81_P10.16mm_Horizontal
- F1: value Fuse -> 1A; footprint Fuse:Fuseholder_Cylinder-6.3x32mm_Schurter_0031-8002_Horizontal_Open -> Fuse:Fuse_Littelfuse_372_D8.50mm
- POTENTIOMETER1: value R_3386P_US -> R_3386P, 100k
- PWR_IN1: value DC005-2.0MM -> DC 2.0mm
- R10, R11, R12, R13, R17, R18, R5, R6: footprint Resistor_THT:R_Axial_DIN0204_L3.6mm_D1.6mm_P7.62mm_Horizontal -> Resistor_THT:R_Axial_DIN0207_L6.3mm_D2.5mm_P7.62mm_Horizontal
- R15: value 1k -> 10k; footprint Resistor_THT:R_Axial_DIN0204_L3.6mm_D1.6mm_P7.62mm_Horizontal -> Resistor_THT:R_Axial_DIN0207_L6.3mm_D2.5mm_P7.62mm_Horizontal
- R16: value 1k -> 20k; footprint Resistor_THT:R_Axial_DIN0204_L3.6mm_D1.6mm_P7.62mm_Horizontal -> Resistor_THT:R_Axial_DIN0207_L6.3mm_D2.5mm_P7.62mm_Horizontal
- R19: value 1k -> 2k; footprint Resistor_THT:R_Axial_DIN0204_L3.6mm_D1.6mm_P7.62mm_Horizontal -> Resistor_THT:R_Axial_DIN0207_L6.3mm_D2.5mm_P7.62mm_Horizontal
- SWITCH1: footprint Button_Switch_THT:SW_Slide_SPDT_Straight_CK_OS102011MS2Q -> Button_Switch_THT:SW_Slide-03_Wuerth-WS-SLTV_10x2.5x6.4_P2.54mm
- moved PWR_IN1 90.9 mm to (99.2, 27.6)
- moved BUZZER1 90.6 mm to (89.6, 72.6), turned to 180 degrees
- moved C12 83.8 mm to (102.1, 92.9), turned to 90 degrees
- moved 1N914 82.5 mm to (74.2, 75.3), turned to 0 degrees
- moved C3 77.0 mm to (120.7, 58.0), turned to 180 degrees
- moved BATTERY1 75.3 mm to (121.4, 25.2), turned to 0 degrees
- moved Q1 74.9 mm to (73.3, 68.3)
- moved D1 74.5 mm to (118.7, 35.0), turned to 180 degrees
- moved C9 71.8 mm to (124.5, 79.2)
- moved LED1 71.2 mm to (131.7, 25.8), turned to 0 degrees
- moved C8 71.2 mm to (124.5, 72.8)
- moved R12 70.7 mm to (66.2, 66.2)
- moved C7 70.7 mm to (124.5, 66.4)
- moved REG1 68.9 mm to (109.8, 49.6)
- moved GYRO1 64.2 mm to (76.1, 52.1)
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Connections:
- BUZZER1 pad 2: Net-(1N914-K) -> Net-(1N914-A)
- C11 pad 1: BattSignal -> GND
- C11 pad 2: GND -> BattSignal
- C12 pad 2: Net-(1N914-K) -> Net-(1N914-A)
- MCU1 pad 25: MIC_SD -> unconnected-(MCU1-GPIO19/USB_D--Pad25)
- MCU1 pad 26: MIC_SCK -> unconnected-(MCU1-GPIO20/USB_D+-Pad26)
- MCU1 pad 27: MIC_WS -> unconnected-(MCU1-GPIO21-Pad27)
- OPAMP1 pad 1: BattSignal -> Net-(OPAMP1A--)
- OPAMP1 pad 2: BattSignal -> Net-(OPAMP1A--)
- OPAMP1 pad 4: (no net) -> GND
- OPAMP1 pad 8: (no net) -> 5V
- OPAMP2 pad 2: GND -> Net-(OPAMP2A--)
- OPAMP2 pad 4: (no net) -> GND
- OPAMP2 pad 8: (no net) -> 5V
- POTENTIOMETER1 pad 2: GND -> Net-(OPAMP2A--)
- POTENTIOMETER1 pad 3: (no net) -> GND
- PWR_IN1 pad 3: (no net) -> unconnected-(PWR_IN1-Pad3)
- Q1 pad 1: Net-(1N914-K) -> Net-(1N914-A)
- R1 pad 1: 8V5 -> Net-(LED1-A)
- R1 pad 2: Net-(LED1-A) -> 8V5
- R17 pad 2: GND -> Net-(OPAMP2A--)
- R4 pad 1: GND -> Net-(OPAMP1A--)
- REG1 pad 1: Net-(LED1-A) -> 8V5
Routing:
- net 5V: track 325.8 -> 171.8 mm
- net 3V3: track 318.4 -> 172.1 mm
- net BUZZER: track 171.0 -> 35.6 mm
- net BattSignal: track 178.8 -> 86.8 mm, vias 0 -> 2
- net MIC_SD: track 90.1 -> 0.00 mm
- net MIC_WS: track 75.3 -> 0.00 mm
- net MIC_SCK: track 71.7 -> 0.00 mm
- net MPU_SCL: track 76.5 -> 13.8 mm
- net MPU_INT: track 80.6 -> 20.5 mm, vias 0 -> 1
- net MPU_SDA: track 73.8 -> 13.8 mm
- net Net-(MK1-+): track 20.9 -> 76.8 mm
- net Net-(1N914-K): track 48.7 -> 0.00 mm
- net Net-(OPAMP2A--): track 0.00 -> 47.5 mm
- net Net-(1N914-A): track 0.00 -> 41.4 mm
- net Net-(OPAMP1A--): track 0.00 -> 32.9 mm, vias 0 -> 1
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Other:
- board outline added: 125.2 x 86.4 mm
