File: embedded_system_project_kicad/embedded_system_project.kicad_sch (KiCad schematic)
At the start: 56 parts, among them Q1 2N2222A, U1 AMS1117CD-3.3

Commit message: Updated repo
Parts:
- removed D1: 1N4007W, Diode_SMD:D_1206_3216Metric_Pad1.42x1.75mm_HandSolder, symbol Device:D
- removed MIC1: INMP441, inmp441:inmp441, symbol inmp441:INMP441
- removed PWR_IN1: DC005-2.0MM, Connector_BarrelJack:BarrelJack_Horizontal, symbol Connector:Barrel_Jack
- removed U1: AMS1117CD-3.3, Package_TO_SOT_SMD:TO-252-3_TabPin2, symbol Regulator_Linear:AMS1117CD-3.3
- added C14: 1000 microF, Capacitor_THT:CP_Axial_L10.0mm_D4.5mm_P15.00mm_Horizontal, symbol Device:C_Polarized
- added D1: 1N4007, Diode_THT:D_DO-41_SOD81_P10.16mm_Horizontal, symbol Diode:1N4007
- added PWR_IN1: DC 2.0mm, Connector_BarrelJack:BarrelJack_Horizontal, symbol Connector:Barrel_Jack_Switch
- added R14: 1k, Resistor_THT:R_Axial_DIN0207_L6.3mm_D2.5mm_P7.62mm_Horizontal, symbol Device:R
- added REG2: LM1085-3.3, LM1085IT-3.3:TO254P1054X470X1955-3, symbol Regulator_Linear:LM1085-3.3
- 1N914: value D -> D2; footprint Diode_THT:D_5KPW_P12.70mm_Horizontal -> 1N914:DIOAD753W49L380D172B
- F1: value Fuse -> 1A; footprint Fuse:Fuseholder_Cylinder-6.3x32mm_Schurter_0031-8002_Horizontal_Open -> Fuse:Fuse_Littelfuse_372_D8.50mm
- POTENTIOMETER1: value R_3386P_US -> R_3386P, 100k
- R10, R11, R12, R13, R17, R18, R5, R6: footprint Resistor_THT:R_Axial_DIN0204_L3.6mm_D1.6mm_P7.62mm_Horizontal -> Resistor_THT:R_Axial_DIN0207_L6.3mm_D2.5mm_P7.62mm_Horizontal
- R15: value 1k -> 10k; footprint Resistor_THT:R_Axial_DIN0204_L3.6mm_D1.6mm_P7.62mm_Horizontal -> Resistor_THT:R_Axial_DIN0207_L6.3mm_D2.5mm_P7.62mm_Horizontal
- R16: value 1k -> 20k; footprint Resistor_THT:R_Axial_DIN0204_L3.6mm_D1.6mm_P7.62mm_Horizontal -> Resistor_THT:R_Axial_DIN0207_L6.3mm_D2.5mm_P7.62mm_Horizontal
- R19: value 1k -> 2k; footprint Resistor_THT:R_Axial_DIN0204_L3.6mm_D1.6mm_P7.62mm_Horizontal -> Resistor_THT:R_Axial_DIN0207_L6.3mm_D2.5mm_P7.62mm_Horizontal
- SWITCH1: footprint Button_Switch_THT:SW_Slide_SPDT_Straight_CK_OS102011MS2Q -> Button_Switch_THT:SW_Slide-03_Wuerth-WS-SLTV_10x2.5x6.4_P2.54mm
Connections:
- net 3V3: now also REG2.2 (VO)
- net 5V: now also 1N914.1 (K), C14.1, R14.2
- net 8V5: now also R1.2, REG1.1 (IN), REG2.3 (VI); no longer R1.1
- net BattSignal: now also C11.2; no longer C11.1, OPAMP1.1, OPAMP1.2 (-)
- net GND: now also C11.1, C14.2, PWR_IN1.2, REG2.1 (GND); no longer 1N914.2 (A), C11.2, OPAMP2.2 (-), POTENTIOMETER1.2, R17.2, R4.1
- net at BATTERY1.1 (Pin_1), F1.1: now also D1.1 (K)
- net at BUZZER1.2 (-), C12.2, Q1.1 (C): now also 1N914.2 (A), R14.1; no longer 1N914.1 (K)
- net MIC_SCK: no longer names the net of MCU1.26 (GPIO20/USB_D+)
- net MIC_SD: no longer names the net of MCU1.25 (GPIO19/USB_D-)
- net MIC_WS: no longer names the net of MCU1.27 (GPIO21)
- new net: LED1.2 (A), R1.1
- new net: OPAMP1.1, OPAMP1.2 (-), R4.1
- new net: OPAMP2.2 (-), POTENTIOMETER1.2, R17.2
- new net: D1.2 (A), PWR_IN1.1
- no-connect marks 1 -> 0
Other:
- note added: "Bypass capacitor (?)"
- note added: "Gain = 1 + R17/R_pot"
- note added: "Gain_min = 1 + 1M/100k = 11 (with potentiometer maxed) -> 11 * 0.2V = 2.2V with example signal of 200mV when clapping"
- note added: "U = R * I = 1k * 2mA = 2V -> safe for red LEDs (2.0 - 2.2V)"
- note added: "V_+ = 8.5 * (5 / (8.6 + 5)) ≈ 3.06 V"
- note added: "V_MIC_ADC = 5 * (2 / (1 + 2)) V_MIC_ADC = 5 * (2 / 3) V_MIC_ADC = 3.33V (maximum scaled value)"
- note added: "V_MIC_ADC = V_out * (R19 / (R18 + R19))"
- note added: "V_out = 5 * (10 / (20 + 10)) V_out = 5 * (10 / 30) V_out = 5 * 0.333 V_out ≈ 1.67V"
- note added: "V_out = 5V (maximum output of the op-amp)"
- note added: "V_out = V_in * (R_lower / (R_upper + R_lower))"
- note added: "f_c = 1 / (2 * π * 10^4 * 100 * 10^-9) ≈ 159.15 Hz"
- moved on the sheet: 1N914, BUZZER1, C10, C11, C12, Q1, R12, R4
